File: HW 2/me433.sch (EAGLE design)
At the start: 21 parts, among them J1 USB_MINI-B_SMT, J2 PIC_ICSP_MINI_5_PIN

Commit message: Gerber Files Generated
Pushing HW 3 andthe generated gerber files.
Parts:
- removed LED4: GREEN, ME433:LED
- added GREEN: (no value), ME433:LED3MM
- added U$6: SLIDE-SWITCH, ME433:SLIDE-SWITCH
- J1: value USB_MINI-B_SMT -> USB_MINI-B; device SparkFun-Connectors:USB_MINI-B_SMT -> ME433:USB_MINI-B
- renumbered LED1 to RED
Connections:
- new net N$16: J1.VBUS, U$6.A
- net GND: now also GREEN.C, U$6.GND; no longer LED4.C
- net N$4: now also U$6.B; no longer J1.VBUS
- net N$9: now also GREEN.A; no longer LED4.A
Other:
- moved on the sheet: J1, J4
